File: Radio PCB/MD9600 Radio.brd (EAGLE design)
At the start: 80 x 32 mm, 14 parts

Commit message: Update PCBs
Parts:
- added E$2: (no value), microchip:SOT23-6
Routing:
- net S$29: track 0.00 -> 29.0 mm
- net S$32: track 0.00 -> 27.1 mm, vias 0 -> 2
- net S$18: track 93.0 -> 67.4 mm
- net S$31: track 0.00 -> 4.00 mm
- net GND: track 28.5 -> 31.0 mm, vias 19 -> 20
Changed lines of the file:
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@@
 <wire x1="57.25" y1="8" x2="79" y2="8" width="0.254" layer="51"/>
 <wire x1="0" y1="32" x2="22" y2="32" width="0" layer="20"/>
+<rectangle x1="52.25" y1="5.5" x2="53.125" y2="6.25" layer="48"/>
 </plain>
 <attributes>
@@
 <element name="R4" library="resistor" package="C0805K" value="SOT" x="43.75" y="6.5" smashed="yes" rot="R90"/>
 <element name="R5" library="resistor" package="C0805K" value="SOT" x="46" y="6.5" smashed="yes" rot="R270"/>
+<element name="E$2" library="microchip" package="SOT23-6" value="" x="54" y="4" smashed="yes" rot="R270">
+<attribute name="VALUE" x="51.328" y="5.397" size="1.016" layer="27" ratio="10" rot="R270"/>
+</element>
 </elements>
 <signals>
@@
 <wire x1="24.75" y1="4.75" x2="31.5" y2="4.75" width="1.27" layer="1"/>
 <via x="51.5" y="8" extent="1-16" drill="0.5" diameter="0.254" shape="octagon"/>
+<via x="56.5" y="2" extent="1-16" drill="0.5" diameter="0.254" shape="octagon"/>
+<wire x1="55" y1="3" x2="56.5" y2="3" width="0.6096" layer="1"/>
+<wire x1="56.5" y1="3" x2="56.5" y2="2" width="0.6096" layer="1"/>
 <wire x1="29.5" y1="4.75" x2="31.5" y2="4.75" width="0" layer="19" extent="1-1"/>
 </signal>
@@
 <wire x1="63.75" y1="13.5" x2="60.125" y2="13.5" width="0.254" layer="1"/>
 <wire x1="60.125" y1="13.5" x2="58.125" y2="13.5" width="0.6096" layer="1"/>
-<wire x1="58.125" y1="13.5" x2="58" y2="2" width="0.6096" layer="1"/>
-<wire x1="58" y1="2" x2="29.75" y2="2" width="0.6096" layer="1"/>
-<wire x1="50.375" y1="7" x2="50.375" y2="1.875" width="0.254" layer="1"/>
-<wire x1="58" y1="2" x2="50.375" y2="1.875" width="0" layer="19" extent="1-1"/>
+<wire x1="58.125" y1="13.5" x2="58" y2="5" width="0.6096" layer="1"/>
+<wire x1="58" y1="5" x2="55" y2="5" width="0.6096" layer="1"/>
+<wire x1="50.375" y1="7" x2="58.125" y2="7" width="0.254" layer="1"/>
+<wire x1="58.125" y1="7" x2="58" y2="5" width="0" layer="19" extent="1-1"/>
 </signal>
 <signal name="S$6">
@@
 <wire x1="50.25" y1="8" x2="51.5" y2="8" width="0.254" layer="1"/>
 </signal>
+<signal name="S$29">
+<wire x1="53" y1="5" x2="50" y2="5" width="0.6096" layer="1"/>
+<wire x1="50" y1="5" x2="50" y2="4" width="0.6096" layer="1"/>
+<wire x1="50" y1="4" x2="50" y2="2" width="0.6096" layer="1"/>
+<wire x1="50" y1="2" x2="30" y2="2" width="0.6096" layer="1"/>
+<wire x1="53" y1="4" x2="50" y2="4" width="0.6096" layer="1"/>
+</signal>
+<signal name="S$31">
+<wire x1="55.125" y1="4" x2="58" y2="4" width="0.6096" layer="1"/>
+<wire x1="58" y1="4" x2="58" y2="5.125" width="0.6096" layer="1"/>
+</signal>
+<signal name="S$32">
+<wire x1="40.5" y1="16.625" x2="40.5" y2="14" width="0.254" layer="1"/>
+<wire x1="40.5" y1="14" x2="45" y2="14" width="0.254" layer="16"/>
+<wire x1="45" y1="14" x2="45" y2="2.5" width="0.254" layer="16"/>
+<wire x1="45" y1="2.5" x2="51.25" y2="2.5" width="0.254" layer="16"/>
+<wire x1="51.25" y1="2.5" x2="51.25" y2="3" width="0.254" layer="1"/>
+<wire x1="51.25" y1="3" x2="53" y2="3" width="0.254" layer="1"/>
+<via x="40.5" y="14" extent="1-16" drill="0.5" diameter="0.254" shape="octagon"/>
+<via x="51.25" y="2.5" extent="1-16" drill="0.5" diameter="0.254" shape="octagon"/>
+</signal>
 </signals>
